File: PCB/kicad/keyboard.kicad_pcb (KiCad board)
At the start: 2 copper layers, 324 x 138 mm, 174 parts

Commit message: Add SK6812-Mini-E LEDs and reroute PCB
Parts:
- added LED1: SK6812MINI-E, PCM_marbastlib-mx:LED_MX_6028R-ROT, B.Cu at (38.1, 43.2)
- added LED10: SK6812MINI-E, PCM_marbastlib-mx:LED_MX_6028R-ROT, B.Cu at (247.7, 43.2)
- added LED11: SK6812MINI-E, PCM_marbastlib-mx:LED_MX_6028R-ROT, B.Cu at (266.7, 43.2)
- added LED12: SK6812MINI-E, PCM_marbastlib-mx:LED_MX_6028R-ROT, B.Cu at (285.8, 43.2)
- added LED13: SK6812MINI-E, PCM_marbastlib-mx:LED_MX_6028R-ROT, B.Cu at (304.8, 43.2)
- added LED14: SK6812MINI-E, PCM_marbastlib-mx:LED_MX_6028R, B.Cu at (333.4, 71.8)
- added LED15: SK6812MINI-E, PCM_marbastlib-mx:LED_MX_6028R, B.Cu at (295.3, 71.8)
- added LED16: SK6812MINI-E, PCM_marbastlib-mx:LED_MX_6028R, B.Cu at (266.7, 71.8)
- added LED17: SK6812MINI-E, PCM_marbastlib-mx:LED_MX_6028R, B.Cu at (247.7, 71.8)
- added LED18: SK6812MINI-E, PCM_marbastlib-mx:LED_MX_6028R, B.Cu at (228.6, 71.8)
- added LED19: SK6812MINI-E, PCM_marbastlib-mx:LED_MX_6028R, B.Cu at (209.6, 71.8)
- added LED2: SK6812MINI-E, PCM_marbastlib-mx:LED_MX_6028R-ROT, B.Cu at (76.2, 43.2)
- added LED20: SK6812MINI-E, PCM_marbastlib-mx:LED_MX_6028R, B.Cu at (190.5, 71.8)
- added LED21: SK6812MINI-E, PCM_marbastlib-mx:LED_MX_6028R, B.Cu at (171.4, 71.8)
- added LED22: SK6812MINI-E, PCM_marbastlib-mx:LED_MX_6028R, B.Cu at (152.4, 71.8)
- added LED23: SK6812MINI-E, PCM_marbastlib-mx:LED_MX_6028R, B.Cu at (133.3, 71.8)
- added LED24: SK6812MINI-E, PCM_marbastlib-mx:LED_MX_6028R, B.Cu at (114.3, 71.8)
- added LED25: SK6812MINI-E, PCM_marbastlib-mx:LED_MX_6028R, B.Cu at (95.2, 71.8)
- added LED26: SK6812MINI-E, PCM_marbastlib-mx:LED_MX_6028R, B.Cu at (76.2, 71.8)
- added LED27: SK6812MINI-E, PCM_marbastlib-mx:LED_MX_6028R, B.Cu at (57.1, 71.8)
- added LED28: SK6812MINI-E, PCM_marbastlib-mx:LED_MX_6028R, B.Cu at (38.1, 71.8)
- added LED29: SK6812MINI-E, PCM_marbastlib-mx:LED_MX_6028R-ROT, B.Cu at (42.9, 90.8)
- added LED3: SK6812MINI-E, PCM_marbastlib-mx:LED_MX_6028R-ROT, B.Cu at (95.2, 43.2)
- added LED30: SK6812MINI-E, PCM_marbastlib-mx:LED_MX_6028R-ROT, B.Cu at (66.7, 90.8)
- added LED31: SK6812MINI-E, PCM_marbastlib-mx:LED_MX_6028R-ROT, B.Cu at (85.7, 90.8)
- added LED32: SK6812MINI-E, PCM_marbastlib-mx:LED_MX_6028R-ROT, B.Cu at (104.8, 90.8)
- added LED33: SK6812MINI-E, PCM_marbastlib-mx:LED_MX_6028R-ROT, B.Cu at (123.8, 90.8)
- added LED34: SK6812MINI-E, PCM_marbastlib-mx:LED_MX_6028R-ROT, B.Cu at (142.9, 90.8)
- added LED35: SK6812MINI-E, PCM_marbastlib-mx:LED_MX_6028R-ROT, B.Cu at (161.9, 90.8)
- added LED36: SK6812MINI-E, PCM_marbastlib-mx:LED_MX_6028R-ROT, B.Cu at (181.0, 90.8)
- added LED37: SK6812MINI-E, PCM_marbastlib-mx:LED_MX_6028R-ROT, B.Cu at (200.0, 90.8)
- added LED38: SK6812MINI-E, PCM_marbastlib-mx:LED_MX_6028R-ROT, B.Cu at (219.1, 90.8)
- added LED39: SK6812MINI-E, PCM_marbastlib-mx:LED_MX_6028R-ROT, B.Cu at (238.1, 90.8)
- added LED4: SK6812MINI-E, PCM_marbastlib-mx:LED_MX_6028R-ROT, B.Cu at (114.3, 43.2)
- added LED40: SK6812MINI-E, PCM_marbastlib-mx:LED_MX_6028R-ROT, B.Cu at (257.2, 90.8)
- added LED41: SK6812MINI-E, PCM_marbastlib-mx:LED_MX_6028R-ROT, B.Cu at (276.2, 90.8)
- added LED42: SK6812MINI-E, PCM_marbastlib-mx:LED_MX_6028R, B.Cu at (297.3, 95.2)
- added LED43: SK6812MINI-E, PCM_marbastlib-mx:LED_MX_6028R-ROT, B.Cu at (333.4, 90.8)
- added LED44: SK6812MINI-E, PCM_marbastlib-mx:LED_MX_6028R, B.Cu at (333.4, 109.9)
- added LED45: SK6812MINI-E, PCM_marbastlib-mx:LED_MX_6028R, B.Cu at (281.0, 109.9)
- added LED46: SK6812MINI-E, PCM_marbastlib-mx:LED_MX_6028R, B.Cu at (261.9, 109.9)
- added LED47: SK6812MINI-E, PCM_marbastlib-mx:LED_MX_6028R, B.Cu at (242.9, 109.9)
- added LED48: SK6812MINI-E, PCM_marbastlib-mx:LED_MX_6028R, B.Cu at (223.8, 109.9)
- added LED49: SK6812MINI-E, PCM_marbastlib-mx:LED_MX_6028R, B.Cu at (204.8, 109.9)
- added LED5: SK6812MINI-E, PCM_marbastlib-mx:LED_MX_6028R-ROT, B.Cu at (133.3, 43.2)
- added LED50: SK6812MINI-E, PCM_marbastlib-mx:LED_MX_6028R, B.Cu at (185.7, 109.9)
- added LED51: SK6812MINI-E, PCM_marbastlib-mx:LED_MX_6028R, B.Cu at (166.7, 109.9)
- added LED52: SK6812MINI-E, PCM_marbastlib-mx:LED_MX_6028R, B.Cu at (147.6, 109.9)
- added LED53: SK6812MINI-E, PCM_marbastlib-mx:LED_MX_6028R, B.Cu at (128.6, 109.9)
- added LED54: SK6812MINI-E, PCM_marbastlib-mx:LED_MX_6028R, B.Cu at (109.5, 109.9)
- added LED55: SK6812MINI-E, PCM_marbastlib-mx:LED_MX_6028R, B.Cu at (90.5, 109.9)
- added LED56: SK6812MINI-E, PCM_marbastlib-mx:LED_MX_6028R, B.Cu at (71.4, 109.9)
- added LED57: SK6812MINI-E, PCM_marbastlib-mx:LED_MX_6028R, B.Cu at (45.2, 109.9)
- added LED58: SK6812MINI-E, PCM_marbastlib-mx:LED_MX_6028R-ROT, B.Cu at (40.5, 128.9)
- added LED59: SK6812MINI-E, PCM_marbastlib-mx:LED_MX_6028R-ROT, B.Cu at (61.9, 128.9)
- added LED6: SK6812MINI-E, PCM_marbastlib-mx:LED_MX_6028R-ROT, B.Cu at (161.9, 43.2)
- added LED60: SK6812MINI-E, PCM_marbastlib-mx:LED_MX_6028R-ROT, B.Cu at (81.0, 128.9)
- added LED61: SK6812MINI-E, PCM_marbastlib-mx:LED_MX_6028R-ROT, B.Cu at (100.0, 128.9)
- added LED62: SK6812MINI-E, PCM_marbastlib-mx:LED_MX_6028R-ROT, B.Cu at (119.1, 128.9)
- added LED63: SK6812MINI-E, PCM_marbastlib-mx:LED_MX_6028R-ROT, B.Cu at (138.1, 128.9)
- added LED64: SK6812MINI-E, PCM_marbastlib-mx:LED_MX_6028R-ROT, B.Cu at (157.2, 128.9)
- added LED65: SK6812MINI-E, PCM_marbastlib-mx:LED_MX_6028R-ROT, B.Cu at (176.2, 128.9)
- added LED66: SK6812MINI-E, PCM_marbastlib-mx:LED_MX_6028R-ROT, B.Cu at (195.3, 128.9)
- added LED67: SK6812MINI-E, PCM_marbastlib-mx:LED_MX_6028R-ROT, B.Cu at (214.3, 128.9)
- added LED68: SK6812MINI-E, PCM_marbastlib-mx:LED_MX_6028R-ROT, B.Cu at (233.4, 128.9)
- added LED69: SK6812MINI-E, PCM_marbastlib-mx:LED_MX_6028R-ROT, B.Cu at (252.4, 128.9)
- added LED7: SK6812MINI-E, PCM_marbastlib-mx:LED_MX_6028R-ROT, B.Cu at (181.0, 43.2)
- added LED70: SK6812MINI-E, PCM_marbastlib-mx:LED_MX_6028R-ROT, B.Cu at (278.6, 128.9)
- added LED71: SK6812MINI-E, PCM_marbastlib-mx:LED_MX_6028R-ROT, B.Cu at (309.6, 133.7)
- added LED72: SK6812MINI-E, PCM_marbastlib-mx:LED_MX_6028R-ROT, B.Cu at (333.4, 128.9)
- added LED73: SK6812MINI-E, PCM_marbastlib-mx:LED_MX_6028R, B.Cu at (328.6, 152.7)
- added LED74: SK6812MINI-E, PCM_marbastlib-mx:LED_MX_6028R, B.Cu at (309.6, 152.7)
- added LED75: SK6812MINI-E, PCM_marbastlib-mx:LED_MX_6028R, B.Cu at (290.5, 152.7)
- added LED76: SK6812MINI-E, PCM_marbastlib-mx:LED_MX_6028R, B.Cu at (266.7, 148.0)
- added LED77: SK6812MINI-E, PCM_marbastlib-mx:LED_MX_6028R, B.Cu at (247.7, 148.0)
- added LED78: SK6812MINI-E, PCM_marbastlib-mx:LED_MX_6028R, B.Cu at (228.6, 148.0)
- added LED79: SK6812MINI-E, PCM_marbastlib-mx:LED_MX_6028R, B.Cu at (159.5, 148.0)
- added LED8: SK6812MINI-E, PCM_marbastlib-mx:LED_MX_6028R-ROT, B.Cu at (200.0, 43.2)
- added LED80: SK6812MINI-E, PCM_marbastlib-mx:LED_MX_6028R, B.Cu at (88.1, 148.0)
- added LED81: SK6812MINI-E, PCM_marbastlib-mx:LED_MX_6028R, B.Cu at (64.3, 148.0)
- added LED82: SK6812MINI-E, PCM_marbastlib-mx:LED_MX_6028R, B.Cu at (40.5, 148.0)
- added LED9: SK6812MINI-E, PCM_marbastlib-mx:LED_MX_6028R-ROT, B.Cu at (219.1, 43.2)
- moved D27 26.0 mm to (268.8, 48.7), turned to -90 degrees
- moved D26 21.5 mm to (252.6, 48.7), turned to -90 degrees
- moved D24 21.2 mm to (210.8, 48.7), turned to -90 degrees
- moved D5 21.0 mm to (136.1, 56.3)
- moved D2 20.4 mm to (84.1, 56.3)
- moved D68 20.3 mm to (201.1, 48.7), turned to -90 degrees
- moved D4 19.8 mm to (119.8, 56.3)
- moved D23 19.7 mm to (191.3, 48.7), turned to -90 degrees
- moved D25 19.6 mm to (233.6, 48.7), turned to -90 degrees
- moved D42 19.5 mm to (272.1, 48.7), turned to -90 degrees
- moved D69 18.7 mm to (223.8, 48.7), turned to -90 degrees
- moved D3 18.6 mm to (103.6, 56.3)
- moved D22 18.1 mm to (175.1, 48.7), turned to -90 degrees
- moved D21 17.0 mm to (158.8, 48.7), turned to -90 degrees
- moved D16 16.6 mm to (67.8, 48.7), turned to -90 degrees
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Connections:
- C_Helios1 pad 13: unconnected-(C_Helios1-5V-Pad13) -> VCC
- C_Helios1 pad 34: unconnected-(C_Helios1-P25-Pad34) -> LED_DIN
Routing:
- net VCC: track 0.00 -> 2606.9 mm, vias 0 -> 10
- net GND: track 365.1 -> 0.00 mm, vias 2 -> 8
- net Net-(LED79-DOUT): track 0.00 -> 66.6 mm
- net LED_DIN: track 0.00 -> 65.3 mm, vias 0 -> 1
- net Net-(LED78-DOUT): track 0.00 -> 64.2 mm
- net Net-(LED44-DOUT): track 0.00 -> 47.6 mm
- net Net-(LED13-DOUT): track 0.00 -> 44.5 mm, vias 0 -> 2
- net Net-(LED42-DOUT): track 0.00 -> 41.5 mm, vias 0 -> 2
- net col13: track 450.1 -> 408.7 mm, vias 1 -> 6
- net col14: track 461.0 -> 424.6 mm, vias 1 -> 6
- net Net-(LED1-DOUT): track 0.00 -> 36.2 mm
- net Net-(LED14-DOUT): track 0.00 -> 33.3 mm
- net Net-(LED72-DOUT): track 0.00 -> 31.2 mm, vias 0 -> 2
- net row1: track 345.6 -> 315.7 mm, vias 14 -> 0
- net row2: track 359.2 -> 330.3 mm, vias 14 -> 16
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- added copper zone on B.Cu, net GND
- added copper zone on F.Cu, net GND
- removed copper zone on B.Cu, net (none)
- removed copper zone on F.Cu, net (none)

Commit message: Add decoupling capacitors
Parts:
- added C1: C, Capacitor_SMD:C_0805_2012Metric_Pad1.18x1.45mm_HandSolder, B.Cu at (29.4, 40.5)
- added C10: C, Capacitor_SMD:C_0805_2012Metric_Pad1.18x1.45mm_HandSolder, B.Cu at (252.9, 42.4)
- added C11: C, Capacitor_SMD:C_0805_2012Metric_Pad1.18x1.45mm_HandSolder, B.Cu at (272.0, 42.4)
- added C12: C, Capacitor_SMD:C_0805_2012Metric_Pad1.18x1.45mm_HandSolder, B.Cu at (291.1, 42.4)
- added C13: C, Capacitor_SMD:C_0805_2012Metric_Pad1.18x1.45mm_HandSolder, B.Cu at (310.0, 42.4)
- added C14: C, Capacitor_SMD:C_0805_2012Metric_Pad1.18x1.45mm_HandSolder, B.Cu at (32.6, 70.7)
- added C15: C, Capacitor_SMD:C_0805_2012Metric_Pad1.18x1.45mm_HandSolder, B.Cu at (65.1, 71.0)
- added C16: C, Capacitor_SMD:C_0805_2012Metric_Pad1.18x1.45mm_HandSolder, B.Cu at (84.3, 71.1)
- added C17: C, Capacitor_SMD:C_0805_2012Metric_Pad1.18x1.45mm_HandSolder, B.Cu at (103.3, 71.0)
- added C18: C, Capacitor_SMD:C_0805_2012Metric_Pad1.18x1.45mm_HandSolder, B.Cu at (122.4, 71.0)
- added C19: C, Capacitor_SMD:C_0805_2012Metric_Pad1.18x1.45mm_HandSolder, B.Cu at (141.5, 71.0)
- added C2: C, Capacitor_SMD:C_0805_2012Metric_Pad1.18x1.45mm_HandSolder, B.Cu at (84.0, 42.5)
- added C20: C, Capacitor_SMD:C_0805_2012Metric_Pad1.18x1.45mm_HandSolder, B.Cu at (160.5, 71.0)
- added C21: C, Capacitor_SMD:C_0805_2012Metric_Pad1.18x1.45mm_HandSolder, B.Cu at (179.6, 71.0)
- added C22: C, Capacitor_SMD:C_0805_2012Metric_Pad1.18x1.45mm_HandSolder, B.Cu at (198.6, 71.0)
- added C23: C, Capacitor_SMD:C_0805_2012Metric_Pad1.18x1.45mm_HandSolder, B.Cu at (217.6, 71.0)
- added C24: C, Capacitor_SMD:C_0805_2012Metric_Pad1.18x1.45mm_HandSolder, B.Cu at (236.7, 71.0)
- added C25: C, Capacitor_SMD:C_0805_2012Metric_Pad1.18x1.45mm_HandSolder, B.Cu at (255.6, 71.0)
- added C26: C, Capacitor_SMD:C_0805_2012Metric_Pad1.18x1.45mm_HandSolder, B.Cu at (275.1, 71.0)
- added C27: C, Capacitor_SMD:C_0805_2012Metric_Pad1.18x1.45mm_HandSolder, B.Cu at (289.1, 72.5)
- added C28: C, Capacitor_SMD:C_0805_2012Metric_Pad1.18x1.45mm_HandSolder, B.Cu at (323.3, 72.5)
- added C29: C, Capacitor_SMD:C_0805_2012Metric_Pad1.18x1.45mm_HandSolder, B.Cu at (52.4, 94.1)
- added C3: C, Capacitor_SMD:C_0805_2012Metric_Pad1.18x1.45mm_HandSolder, B.Cu at (102.1, 42.4)
- added C30: C, Capacitor_SMD:C_0805_2012Metric_Pad1.18x1.45mm_HandSolder, B.Cu at (58.6, 91.5)
- added C31: C, Capacitor_SMD:C_0805_2012Metric_Pad1.18x1.45mm_HandSolder, B.Cu at (77.6, 91.5)
- added C32: C, Capacitor_SMD:C_0805_2012Metric_Pad1.18x1.45mm_HandSolder, B.Cu at (96.8, 91.5)
- added C33: C, Capacitor_SMD:C_0805_2012Metric_Pad1.18x1.45mm_HandSolder, B.Cu at (115.6, 91.5)
- added C34: C, Capacitor_SMD:C_0805_2012Metric_Pad1.18x1.45mm_HandSolder, B.Cu at (134.6, 91.5)
- added C35: C, Capacitor_SMD:C_0805_2012Metric_Pad1.18x1.45mm_HandSolder, B.Cu at (153.6, 91.5)
- added C36: C, Capacitor_SMD:C_0805_2012Metric_Pad1.18x1.45mm_HandSolder, B.Cu at (172.6, 91.5)
- added C37: C, Capacitor_SMD:C_0805_2012Metric_Pad1.18x1.45mm_HandSolder, B.Cu at (191.6, 91.5)
- added C38: C, Capacitor_SMD:C_0805_2012Metric_Pad1.18x1.45mm_HandSolder, B.Cu at (210.6, 91.5)
- added C39: C, Capacitor_SMD:C_0805_2012Metric_Pad1.18x1.45mm_HandSolder, B.Cu at (229.6, 91.5)
- added C4: C, Capacitor_SMD:C_0805_2012Metric_Pad1.18x1.45mm_HandSolder, B.Cu at (121.1, 42.4)
- added C40: C, Capacitor_SMD:C_0805_2012Metric_Pad1.18x1.45mm_HandSolder, B.Cu at (248.6, 91.5)
- added C41: C, Capacitor_SMD:C_0805_2012Metric_Pad1.18x1.45mm_HandSolder, B.Cu at (267.6, 91.5)
- added C42: C, Capacitor_SMD:C_0805_2012Metric_Pad1.18x1.45mm_HandSolder, B.Cu at (291.6, 93.8)
- added C43: C, Capacitor_SMD:C_0805_2012Metric_Pad1.18x1.45mm_HandSolder, B.Cu at (326.9, 95.2)
- added C44: C, Capacitor_SMD:C_0805_2012Metric_Pad1.18x1.45mm_HandSolder, B.Cu at (34.1, 110.0)
- added C45: C, Capacitor_SMD:C_0805_2012Metric_Pad1.18x1.45mm_HandSolder, B.Cu at (79.9, 109.1)
- added C46: C, Capacitor_SMD:C_0805_2012Metric_Pad1.18x1.45mm_HandSolder, B.Cu at (99.0, 109.1)
- added C47: C, Capacitor_SMD:C_0805_2012Metric_Pad1.18x1.45mm_HandSolder, B.Cu at (118.0, 109.1)
- added C48: C, Capacitor_SMD:C_0805_2012Metric_Pad1.18x1.45mm_HandSolder, B.Cu at (137.1, 109.1)
- added C49: C, Capacitor_SMD:C_0805_2012Metric_Pad1.18x1.45mm_HandSolder, B.Cu at (156.1, 109.1)
- added C5: C, Capacitor_SMD:C_0805_2012Metric_Pad1.18x1.45mm_HandSolder, B.Cu at (138.6, 42.4)
- added C50: C, Capacitor_SMD:C_0805_2012Metric_Pad1.18x1.45mm_HandSolder, B.Cu at (175.2, 109.1)
- added C51: C, Capacitor_SMD:C_0805_2012Metric_Pad1.18x1.45mm_HandSolder, B.Cu at (194.2, 109.1)
- added C52: C, Capacitor_SMD:C_0805_2012Metric_Pad1.18x1.45mm_HandSolder, B.Cu at (213.3, 109.1)
- added C53: C, Capacitor_SMD:C_0805_2012Metric_Pad1.18x1.45mm_HandSolder, B.Cu at (232.3, 109.1)
- added C54: C, Capacitor_SMD:C_0805_2012Metric_Pad1.18x1.45mm_HandSolder, B.Cu at (251.4, 109.1)
- added C55: C, Capacitor_SMD:C_0805_2012Metric_Pad1.18x1.45mm_HandSolder, B.Cu at (270.4, 109.1)
- added C56: C, Capacitor_SMD:C_0805_2012Metric_Pad1.18x1.45mm_HandSolder, B.Cu at (300.0, 110.6)
- added C57: C, Capacitor_SMD:C_0805_2012Metric_Pad1.18x1.45mm_HandSolder, B.Cu at (321.5, 110.7)
- added C58: C, Capacitor_SMD:C_0805_2012Metric_Pad1.18x1.45mm_HandSolder, B.Cu at (52.4, 132.5)
- added C59: C, Capacitor_SMD:C_0805_2012Metric_Pad1.18x1.45mm_HandSolder, B.Cu at (73.8, 132.5)
- added C6: C, Capacitor_SMD:C_0805_2012Metric_Pad1.18x1.45mm_HandSolder, B.Cu at (186.1, 42.4)
- added C60: C, Capacitor_SMD:C_0805_2012Metric_Pad1.18x1.45mm_HandSolder, B.Cu at (90.5, 132.5)
- added C61: C, Capacitor_SMD:C_0805_2012Metric_Pad1.18x1.45mm_HandSolder, B.Cu at (100.0, 133.0)
- added C62: C, Capacitor_SMD:C_0805_2012Metric_Pad1.18x1.45mm_HandSolder, B.Cu at (128.6, 132.5)
- added C63: C, Capacitor_SMD:C_0805_2012Metric_Pad1.18x1.45mm_HandSolder, B.Cu at (147.6, 132.5)
- added C64: C, Capacitor_SMD:C_0805_2012Metric_Pad1.18x1.45mm_HandSolder, B.Cu at (167.9, 132.5)
- added C65: C, Capacitor_SMD:C_0805_2012Metric_Pad1.18x1.45mm_HandSolder, B.Cu at (185.7, 132.5)
- added C66: C, Capacitor_SMD:C_0805_2012Metric_Pad1.18x1.45mm_HandSolder, B.Cu at (204.8, 132.5)
- added C67: C, Capacitor_SMD:C_0805_2012Metric_Pad1.18x1.45mm_HandSolder, B.Cu at (223.8, 132.5)
- added C68: C, Capacitor_SMD:C_0805_2012Metric_Pad1.18x1.45mm_HandSolder, B.Cu at (242.9, 132.5)
- added C69: C, Capacitor_SMD:C_0805_2012Metric_Pad1.18x1.45mm_HandSolder, B.Cu at (261.9, 132.5)
- added C7: C, Capacitor_SMD:C_0805_2012Metric_Pad1.18x1.45mm_HandSolder, B.Cu at (205.2, 42.4)
- added C70: C, Capacitor_SMD:C_0805_2012Metric_Pad1.18x1.45mm_HandSolder, B.Cu at (288.1, 132.5)
- added C71: C, Capacitor_SMD:C_0805_2012Metric_Pad1.18x1.45mm_HandSolder, B.Cu at (300.0, 136.9)
- added C72: C, Capacitor_SMD:C_0805_2012Metric_Pad1.18x1.45mm_HandSolder, B.Cu at (323.9, 132.5)
- added C73: C, Capacitor_SMD:C_0805_2012Metric_Pad1.18x1.45mm_HandSolder, B.Cu at (52.4, 144.4)
- added C74: C, Capacitor_SMD:C_0805_2012Metric_Pad1.18x1.45mm_HandSolder, B.Cu at (73.8, 144.4)
- added C75: C, Capacitor_SMD:C_0805_2012Metric_Pad1.18x1.45mm_HandSolder, B.Cu at (97.6, 144.4)
- added C76: C, Capacitor_SMD:C_0805_2012Metric_Pad1.18x1.45mm_HandSolder, B.Cu at (169.1, 144.4)
- added C77: C, Capacitor_SMD:C_0805_2012Metric_Pad1.18x1.45mm_HandSolder, B.Cu at (236.9, 144.4)
- added C78: C, Capacitor_SMD:C_0805_2012Metric_Pad1.18x1.45mm_HandSolder, B.Cu at (256.0, 144.4)
- added C79: C, Capacitor_SMD:C_0805_2012Metric_Pad1.18x1.45mm_HandSolder, B.Cu at (275.0, 144.4)
- added C8: C, Capacitor_SMD:C_0805_2012Metric_Pad1.18x1.45mm_HandSolder, B.Cu at (167.4, 42.4)
- added C80: C, Capacitor_SMD:C_0805_2012Metric_Pad1.18x1.45mm_HandSolder, B.Cu at (298.9, 149.2)
- added C81: C, Capacitor_SMD:C_0805_2012Metric_Pad1.18x1.45mm_HandSolder, B.Cu at (317.9, 149.2)
- added C82: C, Capacitor_SMD:C_0805_2012Metric_Pad1.18x1.45mm_HandSolder, B.Cu at (340.5, 150.3)
- added C83: C, Capacitor_SMD:C_1206_3216Metric_Pad1.33x1.80mm_HandSolder, F.Cu at (62.3, 31.7)
- added C9: C, Capacitor_SMD:C_0805_2012Metric_Pad1.18x1.45mm_HandSolder, B.Cu at (224.3, 42.4)
- added R1: R, Resistor_THT:R_Axial_DIN0207_L6.3mm_D2.5mm_P10.16mm_Horizontal, B.Cu at (62.1, 45.7)
Connections:
- C_Helios1 pad 34: LED_DIN -> Net-(C_Helios1-P25)
Routing:
- net VCC: track 2606.9 -> 2620.3 mm
- net Net-(C_Helios1-P25): track 0.00 -> 10.1 mm
- net row1: track 315.7 -> 307.1 mm
- net row0: track 323.0 -> 315.8 mm
- net GND: track 0.00 -> 6.88 mm, vias 8 -> 38
- net col7: track 219.2 -> 213.2 mm
- net Net-(D36-A): track 26.7 -> 30.7 mm
- net Net-(D75-A): track 87.1 -> 91.0 mm
- net Net-(D34-A): track 26.4 -> 29.9 mm
- net col11: track 348.0 -> 344.8 mm
- net col12: track 369.2 -> 372.3 mm
- net col6: track 221.9 -> 218.8 mm
- net Net-(D67-A): track 72.6 -> 75.6 mm
- net Net-(D68-A): track 71.4 -> 74.4 mm
- net Net-(D69-A): track 71.4 -> 74.2 mm
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